Commit message: Correct urdf model

File: raspigibbon_description/urdf/link.urdf.xacro (robot description, xacro)
@@ -11,5 +11,4 @@
       <insert_block name="joint_origin" />
       <insert_block name="joint_axis" />
-      <!-- <limit lower="&#45;1.57" upper="1.57" effort="0.5293" velocity="6.159937255" /> -->
       <insert_block name="joint_limit" />
       <friction friction="${joint_friction}" />
@@ -50,10 +49,10 @@
       <visual>
         <geometry>
-          <mesh filename="package://raspigibbon_description/meshes/dae/hand${meshid}_link.dae" />
+          <mesh filename="package://raspigibbon_description/meshes/dae/hand_link${meshid}.dae" />
         </geometry>
       </visual>
       <collision>
         <geometry>
-          <mesh filename="package://raspigibbon_description/meshes/dae/hand${meshid}_link.dae" />
+          <mesh filename="package://raspigibbon_description/meshes/dae/hand_link${meshid}.dae" />
         </geometry>
       </collision>

File: raspigibbon_description/urdf/raspigibbon.urdf.xacro (robot description, xacro)
@@ -5,63 +5,63 @@
        xmlns:interface="http://playerstage.sourceforge.net/gazebo/xmlschema/#interface"
        xmlns:xacro="http://ros.org/wiki/xacro">
-  <xacro:include filename="$(find raspigibbon_description)/urdf/base.urdf.xacro" />
-  <xacro:include filename="$(find raspigibbon_description)/urdf/link.urdf.xacro" />
+  <xacro:include filename="$(find raspigibbon_description)/urdf/base.urdf.xacro"/>
+  <xacro:include filename="$(find raspigibbon_description)/urdf/link.urdf.xacro"/>
   <!-- ========== Link & Joint ========== -->
-  <xacro:base_link />
+  <xacro:base_link/>
   <xacro:servo_link linkid="1" meshid="2" jointname="joint1" parent="link0">
-    <origin xyz="0 0 0" rpy="0 0 0" />
-    <axys xyz="0 0 0" />
-    <limit lower="-2.61799387791667" upper="2.61799387791667" effort="0.5293" velocity="6.159937255" />
-    <origin xyz="0.000157 0 0.019222 " />
-    <mass value="0.023032" />
-    <inertia ixx="0.000003514815" ixy="-0.000000000001" iyy="0.000003930066" ixz="-0.000000004487" iyz="0.000000000001" izz="0.000001852796" />
+    <origin xyz="0 0 0.029" rpy="0 0 0"/>
+    <axis xyz="0 0 -1"/>
+    <limit lower="-2.61799387791667" upper="2.61799387791667" effort="0.5293" velocity="6.159937255"/>
+    <origin xyz="0.000157 0 0.019222"/>
+    <mass value="0.023032"/>
+    <inertia ixx="0.000003514815" ixy="-0.000000000001" iyy="0.000003930066" ixz="-0.000000004487" iyz="0.000000000001" izz="0.000001852796"/>
   </xacro:servo_link>
   <xacro:servo_link linkid="2" meshid="3" jointname="joint2" parent="link1">
-    <origin xyz="0 0 0" rpy="0 0 0" />
-    <axys xyz="0 0 0" />
-    <limit lower="-2.61799387791667" upper="2.61799387791667" effort="0.5293" velocity="6.159937255" />
-    <origin xyz="0.000136 0 0.007403 " />
-    <mass value="0.032345" />
-    <inertia ixx="0.000017682369" ixy="-0.000000000049" iyy="0.000019757486" ixz="-0.000000000767" iyz="0.000000000197" izz="0.000004109466" />
+    <origin xyz="0 0 0.02955" rpy="0 0 0"/>
+    <axis xyz="1 0 0"/>
+    <limit lower="-2.61799387791667" upper="2.61799387791667" effort="0.5293" velocity="6.159937255"/>
+    <origin xyz="0.000136 0 0.007403"/>
+    <mass value="0.032345"/>
+    <inertia ixx="0.000017682369" ixy="-0.000000000049" iyy="0.000019757486" ixz="-0.000000000767" iyz="0.000000000197" izz="0.000004109466"/>
   </xacro:servo_link>
   <xacro:servo_link linkid="3" meshid="4" jointname="joint3" parent="link2">
-    <origin xyz="0 0 0" rpy="0 0 0" />
-    <axys xyz="0 0 0" />
-    <limit lower="-2.61799387791667" upper="2.61799387791667" effort="0.5293" velocity="6.159937255" />
-    <origin xyz="0.000136 0 0.007403 " />
-    <mass value="0.032345" />
-    <inertia ixx="0.000017682369" ixy="-0.000000000049" iyy="0.000019757486" ixz="-0.000000000767" iyz="0.000000000197" izz="0.000004109466" />
+    <origin xyz="0 0 0.07655" rpy="0 0 0"/>
+    <axis xyz="1 0 0"/>
+    <limit lower="-2.61799387791667" upper="2.61799387791667" effort="0.5293" velocity="6.159937255"/>
+    <origin xyz="0.000136 0 0.007403"/>
+    <mass value="0.032345"/>
+    <inertia ixx="0.000017682369" ixy="-0.000000000049" iyy="0.000019757486" ixz="-0.000000000767" iyz="0.000000000197" izz="0.000004109466"/>
   </xacro:servo_link>
   <xacro:servo_link linkid="4" meshid="5" jointname="joint4" parent="link3">
-    <origin xyz="0 0 0" rpy="0 0 0" />
-    <axys xyz="0 0 0" />
-    <limit lower="-2.61799387791667" upper="2.61799387791667" effort="0.5293" velocity="6.159937255" />
-    <origin xyz="0.000253 0.000821 0.013947 " />
-    <mass value="0.041117" />
-    <inertia ixx="0.000006913101" ixy="0.000000054083" iyy="0.000009528465" ixz="-0.000000059992" iyz="-0.000000095617" izz="0.000008648857" />
+    <origin xyz="0 0 0.07655" rpy="0 0 0"/>
+    <axis xyz="1 0 0"/>
+    <limit lower="-2.61799387791667" upper="2.61799387791667" effort="0.5293" velocity="6.159937255"/>
+    <origin xyz="0.000253 0.000821 0.013947"/>
+    <mass value="0.041117"/>
+    <inertia ixx="0.000006913101" ixy="0.000000054083" iyy="0.000009528465" ixz="-0.000000059992" iyz="-0.000000095617" izz="0.000008648857"/>
   </xacro:servo_link>
   <xacro:hand_link linkid="5" meshid="1" jointname="joint5" parent="link4">
-    <origin xyz="0 0 0" rpy="0 0 0" />
-    <axys xyz="0 0 0" />
-    <limit lower="-2.61799387791667" upper="2.61799387791667" effort="0.5293" velocity="6.159937255" />
-    <origin xyz="0.000253 0.000821 0.013947 " />
-    <mass value="0.041117" />
-    <inertia ixx="0.000006913101" ixy="0.000000054083" iyy="0.000009528465" ixz="-0.000000059992" iyz="-0.000000095617" izz="0.000008648857" />
+    <origin xyz="-0.0091 0 0.0342" rpy="0 -1.5708 -1.5708"/>
+    <axis xyz="0 0 1"/>
+    <limit lower="-2.61799387791667" upper="2.61799387791667" effort="0.5293" velocity="6.159937255"/>
+    <origin xyz="0.000253 0.000821 0.013947"/>
+    <mass value="0.041117"/>
+    <inertia ixx="0.000006913101" ixy="0.000000054083" iyy="0.000009528465" ixz="-0.000000059992" iyz="-0.000000095617" izz="0.000008648857"/>
   </xacro:hand_link>
   <xacro:hand_link linkid="6" meshid="2" jointname="joint6" parent="link4">
-    <origin xyz="0 0 0" rpy="0 0 0" />
-    <axys xyz="0 0 0" />
-    <limit lower="-2.61799387791667" upper="2.61799387791667" effort="0.5293" velocity="6.159937255" />
-    <origin xyz="0.000253 0.000821 0.013947 " />
-    <mass value="0.041117" />
-    <inertia ixx="0.000006913101" ixy="0.000000054083" iyy="0.000009528465" ixz="-0.000000059992" iyz="-0.000000095617" izz="0.000008648857" />
+    <origin xyz="0.0091 0.0 0.0342" rpy="0 -1.5708 -1.5708"/>
+    <axis xyz="0 0 1"/>
+    <limit lower="-2.61799387791667" upper="2.61799387791667" effort="0.5293" velocity="6.159937255"/>
+    <origin xyz="0.000253 0.000821 0.013947"/>
+    <mass value="0.041117"/>
+    <inertia ixx="0.000006913101" ixy="0.000000054083" iyy="0.000009528465" ixz="-0.000000059992" iyz="-0.000000095617" izz="0.000008648857"/>
   </xacro:hand_link>
   <!-- ========== Transmission ========== -->
-  <xacro:servo_trans joint_name="joint1" interface="PositionJointInterface" />
-  <xacro:servo_trans joint_name="joint2" interface="PositionJointInterface" />
-  <xacro:servo_trans joint_name="joint3" interface="PositionJointInterface" />
-  <xacro:servo_trans joint_name="joint4" interface="PositionJointInterface" />
-  <xacro:servo_trans joint_name="joint5" interface="PositionJointInterface" />
-  <xacro:servo_trans joint_name="joint6" interface="PositionJointInterface" />
+  <xacro:servo_trans joint_name="joint1" interface="PositionJointInterface"/>
+  <xacro:servo_trans joint_name="joint2" interface="PositionJointInterface"/>
+  <xacro:servo_trans joint_name="joint3" interface="PositionJointInterface"/>
+  <xacro:servo_trans joint_name="joint4" interface="PositionJointInterface"/>
+  <xacro:servo_trans joint_name="joint5" interface="PositionJointInterface"/>
+  <xacro:servo_trans joint_name="joint6" interface="PositionJointInterface"/>
   <!-- ========== Gazebo ========== -->
   <gazebo>
@@ -70,5 +70,5 @@
     </plugin>
   </gazebo>
-  <xacro:base_gazebo />
+  <xacro:base_gazebo/>
   <xacro:link_gazebo id="1"/>
   <xacro:link_gazebo id="2"/>
