Commit message: Add xacro files

File: raspigibbon_description/urdf/base.urdf.xacro (robot description, xacro)
@@ -4,5 +4,5 @@
   <xacro:property name="M_PI" value="3.1415926535897931" />
   <xacro:property name="velocity_scale_factor" value="1.0"/>
-  <xacro:macro name="base">
+  <xacro:macro name="base_link">
     <link name="base_link">
       <visual>
@@ -22,4 +22,26 @@
       </inertial>
     </link>
+    <joint name="joint0" type="fixed">
+      <origin xyz="0.0 0.0 0.0" />
+      <parent link="base_link" />
+      <child link="link0" />
+    </joint>
+    <link name="link0">
+      <visual>
+        <geometry>
+          <mesh filename="package://raspigibbon_description/meshes/dae/servo1_link.dae" />
+        </geometry>
+      </visual>
+      <collision>
+        <geometry>
+          <mesh filename="package://raspigibbon_description/meshes/dae/servo1_link.dae" />
+        </geometry>
+      </collision>
+      <inertial>
+        <origin xyz="0 -0.008722 0.01556 " />
+        <mass value="0.022267" />
+        <inertia ixx="0.000003621474" ixy="0.000000000001" iyy="0.000001983132" ixz="-0.000000000001" iyz="-0.000000215045" izz="0.000003182899" />
+      </inertial>
+    </link>
   </xacro:macro>
 </robot>

File: raspigibbon_description/urdf/link.urdf.xacro (robot description, xacro)
@@ -2,7 +2,10 @@
 <robot xmlns:xacro="http://ros.org/wiki/xacro">
   <xacro:include filename="$(find raspigibbon_description)/urdf/link.gazebo.xacro" />
+  <xacro:include filename="$(find raspigibbon_description)/urdf/link.transmission.xacro" />
   <xacro:property name="M_PI" value="3.1415926535897931" />
   <xacro:property name="velocity_scale_factor" value="1.0" />
-  <xacro:macro name="link" params="id jointname parent *joint_origin *joint_axis *joint_limit *inertial_origin *inertial_mass *inertial_inertia">
+  <xacro:property name="joint_friction" value="1.0" />
+  <xacro:property name="joint_damping" value="1.0" />
+  <xacro:macro name="servo_link" params="linkid meshid jointname parent *joint_origin *joint_axis *joint_limit *inertial_origin *inertial_mass *inertial_inertia">
     <joint name="${jointname}" type="revolute">
       <insert_block name="joint_origin" />
@@ -13,15 +16,44 @@
       <dynamics damping="${joint_damping}" />
       <parent link="${parent}" />
-      <child link="link${id}" />
+      <child link="link${linkid}" />
     </joint>
-    <link name="link${id}">
+    <link name="link${linkid}">
       <visual>
         <geometry>
-          <mesh filename="package://raspigibbon_description/meshes/dae/servo${id}_link.dae" />
+          <mesh filename="package://raspigibbon_description/meshes/dae/servo${meshid}_link.dae" />
         </geometry>
       </visual>
       <collision>
         <geometry>
-          <mesh filename="package://raspigibbon_description/meshes/dae/servo${id}_link.dae" />
+          <mesh filename="package://raspigibbon_description/meshes/dae/servo${meshid}_link.dae" />
+        </geometry>
+      </collision>
+      <inertial>
+        <insert_block name="inertial_origin" />
+        <insert_block name="inertial_mass" />
+        <insert_block name="inertial_inertia" />
+      </inertial>
+    </link>
+  </xacro:macro>
+  <xacro:macro name="hand_link" params="linkid meshid jointname parent *joint_origin *joint_axis *joint_limit *inertial_origin *inertial_mass *inertial_inertia">
+    <joint name="${jointname}" type="revolute">
+      <insert_block name="joint_origin" />
+      <insert_block name="joint_axis" />
+      <!-- <limit lower="&#45;1.57" upper="1.57" effort="0.5293" velocity="6.159937255" /> -->
+      <insert_block name="joint_limit" />
+      <friction friction="${joint_friction}" />
+      <dynamics damping="${joint_damping}" />
+      <parent link="${parent}" />
+      <child link="link${linkid}" />
+    </joint>
+    <link name="link${linkid}">
+      <visual>
+        <geometry>
+          <mesh filename="package://raspigibbon_description/meshes/dae/hand${meshid}_link.dae" />
+        </geometry>
+      </visual>
+      <collision>
+        <geometry>
+          <mesh filename="package://raspigibbon_description/meshes/dae/hand${meshid}_link.dae" />
         </geometry>
       </collision>

File: raspigibbon_description/urdf/raspigibbon.urdf.xacro (robot description, xacro)
@@ -8,12 +8,60 @@
   <xacro:include filename="$(find raspigibbon_description)/urdf/link.urdf.xacro" />
   <!-- ========== Link & Joint ========== -->
-  <xacro:>
+  <xacro:base_link />
+  <xacro:servo_link linkid="1" meshid="2" jointname="joint1" parent="link0">
+    <origin xyz="0 0 0" rpy="0 0 0" />
+    <axys xyz="0 0 0" />
+    <limit lower="-2.61799387791667" upper="2.61799387791667" effort="0.5293" velocity="6.159937255" />
+    <origin xyz="0.000157 0 0.019222 " />
+    <mass value="0.023032" />
+    <inertia ixx="0.000003514815" ixy="-0.000000000001" iyy="0.000003930066" ixz="-0.000000004487" iyz="0.000000000001" izz="0.000001852796" />
+  </xacro:servo_link>
+  <xacro:servo_link linkid="2" meshid="3" jointname="joint2" parent="link1">
+    <origin xyz="0 0 0" rpy="0 0 0" />
+    <axys xyz="0 0 0" />
+    <limit lower="-2.61799387791667" upper="2.61799387791667" effort="0.5293" velocity="6.159937255" />
+    <origin xyz="0.000136 0 0.007403 " />
+    <mass value="0.032345" />
+    <inertia ixx="0.000017682369" ixy="-0.000000000049" iyy="0.000019757486" ixz="-0.000000000767" iyz="0.000000000197" izz="0.000004109466" />
+  </xacro:servo_link>
+  <xacro:servo_link linkid="3" meshid="4" jointname="joint3" parent="link2">
+    <origin xyz="0 0 0" rpy="0 0 0" />
+    <axys xyz="0 0 0" />
+    <limit lower="-2.61799387791667" upper="2.61799387791667" effort="0.5293" velocity="6.159937255" />
+    <origin xyz="0.000136 0 0.007403 " />
+    <mass value="0.032345" />
+    <inertia ixx="0.000017682369" ixy="-0.000000000049" iyy="0.000019757486" ixz="-0.000000000767" iyz="0.000000000197" izz="0.000004109466" />
+  </xacro:servo_link>
+  <xacro:servo_link linkid="4" meshid="5" jointname="joint4" parent="link3">
+    <origin xyz="0 0 0" rpy="0 0 0" />
+    <axys xyz="0 0 0" />
+    <limit lower="-2.61799387791667" upper="2.61799387791667" effort="0.5293" velocity="6.159937255" />
+    <origin xyz="0.000253 0.000821 0.013947 " />
+    <mass value="0.041117" />
+    <inertia ixx="0.000006913101" ixy="0.000000054083" iyy="0.000009528465" ixz="-0.000000059992" iyz="-0.000000095617" izz="0.000008648857" />
+  </xacro:servo_link>
+  <xacro:hand_link linkid="5" meshid="1" jointname="joint5" parent="link4">
+    <origin xyz="0 0 0" rpy="0 0 0" />
+    <axys xyz="0 0 0" />
+    <limit lower="-2.61799387791667" upper="2.61799387791667" effort="0.5293" velocity="6.159937255" />
+    <origin xyz="0 0 0" rpy="0 0 0" />
+    <axys xyz="0 0 0" />
+    <limit lower="-2.61799387791667" upper="2.61799387791667" effort="0.5293" velocity="6.159937255" />
+  </xacro:hand_link>
+  <xacro:hand_link linkid="6" meshid="2" jointname="joint6" parent="link4">
+    <origin xyz="0 0 0" rpy="0 0 0" />
+    <axys xyz="0 0 0" />
+    <limit lower="-2.61799387791667" upper="2.61799387791667" effort="0.5293" velocity="6.159937255" />
+    <origin xyz="0 0 0" rpy="0 0 0" />
+    <axys xyz="0 0 0" />
+    <limit lower="-2.61799387791667" upper="2.61799387791667" effort="0.5293" velocity="6.159937255" />
+  </xacro:hand_link>
   <!-- ========== Transmission ========== -->
-  <xacro:transmission prefix="joint1" interface="PositionJointInterface" />
-  <xacro:transmission prefix="joint2" interface="PositionJointInterface" />
-  <xacro:transmission prefix="joint3" interface="PositionJointInterface" />
-  <xacro:transmission prefix="joint4" interface="PositionJointInterface" />
-  <xacro:transmission prefix="joint5" interface="PositionJointInterface" />
-  <xacro:transmission prefix="joint6" interface="PositionJointInterface" />
+  <xacro:servo_trans joint_name="joint1" interface="PositionJointInterface" />
+  <xacro:servo_trans joint_name="joint2" interface="PositionJointInterface" />
+  <xacro:servo_trans joint_name="joint3" interface="PositionJointInterface" />
+  <xacro:servo_trans joint_name="joint4" interface="PositionJointInterface" />
+  <xacro:servo_trans joint_name="joint5" interface="PositionJointInterface" />
+  <xacro:servo_trans joint_name="joint6" interface="PositionJointInterface" />
   <!-- ========== Gazebo ========== -->
   <gazebo>

Commit message: Update to fix base_link to world

File: raspigibbon_description/urdf/base.urdf.xacro (robot description, xacro)
@@ -5,4 +5,9 @@
   <xacro:property name="velocity_scale_factor" value="1.0"/>
   <xacro:macro name="base_link">
+    <link name="world"/>
+    <joint name="world2base" type="fixed">
+      <parent link="world"/>
+      <child link="base_link"/>
+    </joint>
     <link name="base_link">
       <visual>

File: raspigibbon_description/urdf/raspigibbon.urdf (robot description, URDF)
Before this commit: robot raspigibbon, 8 links, 7 joints
Links:
- added link world
Joints:
- added joint world2base: type fixed, parent world, child base_link
