Commit message: Add base link as master fixed link

File: raspigibbon_description/urdf/raspigibbon.urdf (robot description, URDF)
Before this commit: robot raspigibbon, 7 links, 6 joints
Links:
- added link base
Joints:
- added joint joint0: type fixed, parent base, child base_link, origin xyz=0 0 0 rpy=0 0 0

Commit message: Update urdf

File: raspigibbon_description/urdf/raspigibbon.urdf (robot description, URDF)
Before this commit: robot raspigibbon, 8 links, 7 joints
Links:
- removed link base
- added link link0, mass 0.022267; collision mesh filename=package://raspigibbon_description/meshes/dae/servo1_link.dae; visual mesh filename=package://raspigibbon_description/meshes/dae/servo1_link.dae
- link base_link: mass None -> 0.060272; geometry collision mesh filename=package://raspigibbon_description/meshes/dae/base_link.dae; visual mesh filename=package://raspigibbon_description/meshes/dae/base_link.dae
- link link1: mass None -> 0.023032; geometry collision mesh filename=package://raspigibbon_description/meshes/dae/servo2_link.dae; visual mesh filename=package://raspigibbon_description/meshes/dae/servo2_link.dae
- link link2: mass None -> 0.032345; geometry collision mesh filename=package://raspigibbon_description/meshes/dae/servo3_link.dae; visual mesh filename=package://raspigibbon_description/meshes/dae/servo3_link.dae
- link link3: mass None -> 0.032345; geometry collision mesh filename=package://raspigibbon_description/meshes/dae/servo4_link.dae; visual mesh filename=package://raspigibbon_description/meshes/dae/servo4_link.dae
- link link4: mass None -> 0.041117; geometry collision mesh filename=package://raspigibbon_description/meshes/dae/servo5_link.dae; visual mesh filename=package://raspigibbon_description/meshes/dae/servo5_link.dae
- link link5: mass None -> 0.041117; geometry collision mesh filename=package://raspigibbon_description/meshes/dae/hand_link1.dae; visual mesh filename=package://raspigibbon_description/meshes/dae/hand_link1.dae
- link link6: mass None -> 0.041117; geometry collision mesh filename=package://raspigibbon_description/meshes/dae/hand_link2.dae; visual mesh filename=package://raspigibbon_description/meshes/dae/hand_link2.dae
Joints:
- joint joint0: child base_link -> link0; origin xyz=0 0 0 rpy=0 0 0 -> xyz=0.0 0.0 0.0; parent base -> base_link
- joint joint1: axis 0 0 1 -> 0 0 -1; limit lower=-2.61 upper=2.61 effort=0.5 velocity=6.0 -> lower=-2.61799387791667 upper=2.61799387791667 effort=0.5293 velocity=6.159937255; origin xyz=0.0145 0 0.0454 rpy=0 0 0 -> xyz=0 0 0.029 rpy=0 0 0; parent base_link -> link0
- joint joint2: axis 0 1 0 -> 1 0 0; limit lower=-1.75 upper=1.75 effort=0.5 velocity=6.0 -> lower=-2.61799387791667 upper=2.61799387791667 effort=0.5293 velocity=6.159937255; origin xyz=0 0 0.026 rpy=0 0 0 -> xyz=0 0 0.02955 rpy=0 0 0
- joint joint3: axis 0 -1 0 -> 1 0 0; limit lower=-2.55 upper=2.55 effort=0.5 velocity=6.0 -> lower=-2.61799387791667 upper=2.61799387791667 effort=0.5293 velocity=6.159937255; origin xyz=0 0 0.083 rpy=0 0 0 -> xyz=0 0 0.07655 rpy=0 0 0
- joint joint4: axis 0 -1 0 -> 1 0 0; limit lower=-1.80 upper=1.80 effort=0.5 velocity=6.0 -> lower=-2.61799387791667 upper=2.61799387791667 effort=0.5293 velocity=6.159937255; origin xyz=0 0 0.0935 rpy=0 0 0 -> xyz=0 0 0.07655 rpy=0 0 0
- joint joint5: axis -1 0 0 -> 0 0 1; limit lower=-0.69 upper=0.69 effort=0.5 velocity=6.0 -> lower=-2.61799387791667 upper=2.61799387791667 effort=0.5293 velocity=6.159937255; origin xyz=0 -0.0145 0.045 rpy=0 0 0 -> xyz=-0.0091 0 0.0342 rpy=0 -1.5708 -1.5708
- joint joint6: axis -1 0 0 -> 0 0 1; limit lower=-0.69 upper=0.69 effort=0.5 velocity=6.0 -> lower=-2.61799387791667 upper=2.61799387791667 effort=0.5293 velocity=6.159937255; origin xyz=0 0.0145 0.045 rpy=0 0 3.141592 -> xyz=0.0091 0.0 0.0342 rpy=0 -1.5708 -1.5708

Commit message: Correct URDF model

File: raspigibbon_description/urdf/raspigibbon.urdf (robot description, URDF)
Before this commit: robot raspigibbon, 9 links, 8 joints
Joints:
- joint joint1: limit lower=-2.61799387791667 upper=2.61799387791667 effort=0.5293 velocity=6.159937255 -> lower=-2.52 upper=2.52 effort=0.5293 velocity=6.159937255
- joint joint2: limit lower=-2.61799387791667 upper=2.61799387791667 effort=0.5293 velocity=6.159937255 -> lower=-2.52 upper=2.52 effort=0.5293 velocity=6.159937255; origin xyz=0 0 0.02955 rpy=0 0 0 -> xyz=0 0 0.03055 rpy=0 0 0
- joint joint3: limit lower=-2.61799387791667 upper=2.61799387791667 effort=0.5293 velocity=6.159937255 -> lower=-2.52 upper=2.52 effort=0.5293 velocity=6.159937255; origin xyz=0 0 0.07655 rpy=0 0 0 -> xyz=0 0 0.08055 rpy=0 0 0
- joint joint4: limit lower=-2.61799387791667 upper=2.61799387791667 effort=0.5293 velocity=6.159937255 -> lower=-1.99 upper=1.99 effort=0.5293 velocity=6.159937255; origin xyz=0 0 0.07655 rpy=0 0 0 -> xyz=0 0 0.08055 rpy=0 0 0
- joint joint5: limit lower=-2.61799387791667 upper=2.61799387791667 effort=0.5293 velocity=6.159937255 -> lower=-1.92 upper=0.05 effort=0.5293 velocity=6.159937255
- joint joint6: limit lower=-2.61799387791667 upper=2.61799387791667 effort=0.5293 velocity=6.159937255 -> lower=-0.05 upper=1.92 effort=0.5293 velocity=6.159937255

File: raspigibbon_description/urdf/raspigibbon.urdf.xacro (robot description, xacro)
@@ -12,5 +12,5 @@
     <origin xyz="0 0 0.029" rpy="0 0 0"/>
     <axis xyz="0 0 -1"/>
-    <limit lower="-2.61799387791667" upper="2.61799387791667" effort="0.5293" velocity="6.159937255"/>
+    <limit lower="-2.52" upper="2.52" effort="0.5293" velocity="6.159937255"/>
     <origin xyz="0.000157 0 0.019222"/>
     <mass value="0.023032"/>
@@ -18,7 +18,7 @@
   </xacro:servo_link>
   <xacro:servo_link linkid="2" meshid="3" jointname="joint2" parent="link1">
-    <origin xyz="0 0 0.02955" rpy="0 0 0"/>
+    <origin xyz="0 0 0.03055" rpy="0 0 0"/>
     <axis xyz="1 0 0"/>
-    <limit lower="-2.61799387791667" upper="2.61799387791667" effort="0.5293" velocity="6.159937255"/>
+    <limit lower="-2.52" upper="2.52" effort="0.5293" velocity="6.159937255"/>
     <origin xyz="0.000136 0 0.007403"/>
     <mass value="0.032345"/>
@@ -26,7 +26,7 @@
   </xacro:servo_link>
   <xacro:servo_link linkid="3" meshid="4" jointname="joint3" parent="link2">
-    <origin xyz="0 0 0.07655" rpy="0 0 0"/>
+    <origin xyz="0 0 0.08055" rpy="0 0 0"/>
     <axis xyz="1 0 0"/>
-    <limit lower="-2.61799387791667" upper="2.61799387791667" effort="0.5293" velocity="6.159937255"/>
+    <limit lower="-2.52" upper="2.52" effort="0.5293" velocity="6.159937255"/>
     <origin xyz="0.000136 0 0.007403"/>
     <mass value="0.032345"/>
@@ -34,7 +34,7 @@
   </xacro:servo_link>
   <xacro:servo_link linkid="4" meshid="5" jointname="joint4" parent="link3">
-    <origin xyz="0 0 0.07655" rpy="0 0 0"/>
+    <origin xyz="0 0 0.08055" rpy="0 0 0"/>
     <axis xyz="1 0 0"/>
-    <limit lower="-2.61799387791667" upper="2.61799387791667" effort="0.5293" velocity="6.159937255"/>
+    <limit lower="-1.99" upper="1.99" effort="0.5293" velocity="6.159937255"/>
     <origin xyz="0.000253 0.000821 0.013947"/>
     <mass value="0.041117"/>
@@ -44,5 +44,5 @@
     <origin xyz="-0.0091 0 0.0342" rpy="0 -1.5708 -1.5708"/>
     <axis xyz="0 0 1"/>
-    <limit lower="-2.61799387791667" upper="2.61799387791667" effort="0.5293" velocity="6.159937255"/>
+    <limit lower="-1.92" upper="0.05" effort="0.5293" velocity="6.159937255"/>
     <origin xyz="0.000253 0.000821 0.013947"/>
     <mass value="0.041117"/>
@@ -52,5 +52,5 @@
     <origin xyz="0.0091 0.0 0.0342" rpy="0 -1.5708 -1.5708"/>
     <axis xyz="0 0 1"/>
-    <limit lower="-2.61799387791667" upper="2.61799387791667" effort="0.5293" velocity="6.159937255"/>
+    <limit lower="-0.05" upper="1.92" effort="0.5293" velocity="6.159937255"/>
     <origin xyz="0.000253 0.000821 0.013947"/>
     <mass value="0.041117"/>
